File: eagle/atmel_midi_clock.brd (EAGLE design)
At the start: 101 x 80.8 mm, 46 parts, among them IC1 TL084P, IC2 40106N, U1 ATMEGA328P_PDIP, X1 22-23-2031, X2 22-23-2031, X3 22-23-2031, X4 22-23-2031

Commit message: layout begins
Parts:
- removed C7: 100n, rcl:C050-024X044
- removed IC1: TL084P, linear:DIL14
- removed MIDI_IN_4: midi pin 4, wirepad:2,54/0,9
- removed MIDI_IN_5: midi pin 5, wirepad:2,54/0,9
- removed X1, X2, X3, X4: 22-23-2031, con-molex:22-23-2031
- added CLOCK_LED, CONTINUE_LED, START_LED, STOP_LED: (no value), led:LED5MM
- added MIDI_IN: 22-23-2021, con-molex:22-23-2021
- added R16, R17, R18, R19: 330, rcl:0207/10
- added THRU1, THRU2, THRU3, THRU4: 22-23-2031, con-molex:22-23-2031
- moved R15 328.1 mm to (-31.8, 91.4)
- moved R14 323.9 mm to (-19.1, 91.4)
- moved R13 314.3 mm to (-82.5, 86.4)
- moved R11 307.5 mm to (-57.1, 86.4)
- moved R10 303.8 mm to (-44.5, 86.4)
- moved R9 297.7 mm to (-31.8, 86.4)
- moved R7 295.1 mm to (-82.5, 81.3)
- moved R6 287.4 mm to (-69.8, 81.3)
- moved R4 278.5 mm to (-44.5, 81.3)
- moved LED1 264.2 mm to (-21.6, 76.2)
- moved R12 245.2 mm to (-69.8, 86.4)
- moved IC2 227.4 mm to (-43.2, 47.0)
- moved U$1 203.4 mm to (25.4, 35.6), turned to 270 degrees
- moved R8 198.9 mm to (-19.1, 86.4)
- moved R5 154.0 mm to (-57.1, 81.3)
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Connections:
- new net N$37: R17.2, START_LED.A
- new net N$38: CLOCK_LED.A, R16.2
- new net N$39: CONTINUE_LED.A, R18.2
- new net N$40: R19.2, STOP_LED.A
- net +12V: no longer C7.1, IC1.4
- net GND: now also CLOCK_LED.K, CONTINUE_LED.K, START_LED.K, STOP_LED.K, THRU1.2, THRU2.2, THRU3.2, THRU4.2; no longer X1.2, X2.2, X3.2, X4.2
- net N$1: now also R18.1, U1.16; no longer U1.6
- net N$10: now also R17.1, U1.15; no longer U1.5
- net N$26: now also THRU1.1; no longer X1.1
- net N$27: now also THRU2.1; no longer X2.1
- net N$28: now also THRU3.1; no longer X3.1
- net N$29: no longer C7.2, IC1.11
- net N$3: now also MIDI_IN.2; no longer MIDI_IN_5.1
- net N$32: now also THRU4.1; no longer X4.1
- net N$33: now also THRU1.3; no longer X1.3
- net N$34: now also THRU2.3; no longer X2.3
- net N$35: now also THRU3.3; no longer X3.3
- net N$36: now also THRU4.3; no longer X4.3
- net N$6: now also R19.1, U1.17; no longer U1.11
- net N$8: now also MIDI_IN.1; no longer MIDI_IN_4.1
- net N$9: now also R16.1, U1.14; no longer U1.4
Routing:
- net N$29: track 254.4 -> 0.00 mm
- net +5V: track 170.5 -> 0.00 mm
- net N$31: track 143.7 -> 0.00 mm
- net +12V: track 39.0 -> 0.00 mm
- net N$30: track 37.7 -> 0.00 mm
- net N$5: track 13.5 -> 0.00 mm
- net N$4: track 13.1 -> 0.00 mm
- net N$11: track 11.2 -> 0.00 mm
- net N$3: track 10.3 -> 0.00 mm
- net N$7: track 8.90 -> 0.00 mm
- net N$43: track 7.40 -> 0.00 mm
- net N$8: track 4.02 -> 0.00 mm
- net N$19: track 0.65 -> 0.00 mm
Other:
- board size 101 x 80.8 mm -> 100 x 80 mm

Commit message: almost routed
Parts:
- moved R13 167.9 mm to (80.0, 44.5), turned to 90 degrees
- moved MIDI_IN 149.9 mm to (64.8, 73.7), turned to 270 degrees
- moved R7 148.2 mm to (61.0, 44.5), turned to 270 degrees
- moved R11 141.0 mm to (77.5, 44.5), turned to 90 degrees
- moved R1 138.6 mm to (52.1, 66.0), turned to 270 degrees
- moved R6 138.3 mm to (63.5, 44.5), turned to 270 degrees
- moved RST2 133.7 mm to (55.9, 63.5)
- moved RST1 127.8 mm to (55.9, 59.7)
- moved R15 127.6 mm to (77.5, 25.4), turned to 270 degrees
- moved R12 125.7 mm to (39.4, 24.1), turned to 90 degrees
- moved STOP_LED 125.1 mm to (38.1, 35.6)
- moved R10 124.6 mm to (63.5, 24.1), turned to 90 degrees
- moved R19 123.6 mm to (31.8, 44.5)
- moved THRU4 121.3 mm to (71.1, 22.9)
- moved R14 119.1 mm to (80.0, 25.4), turned to 270 degrees
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Connections:
- net N$1: now also U1.17; no longer U1.16
- net N$10: now also U1.16; no longer U1.15
- net N$6: now also U1.18; no longer U1.17
- net N$9: now also U1.15; no longer U1.14

Commit message: routed
Parts:
- moved R16 20.4 mm to (16.5, 34.3), turned to 180 degrees
- moved R17 20.4 mm to (16.5, 26.7)
- moved R7 15.7 mm to (64.8, 29.2), turned to 90 degrees
- moved START_LED 14.0 mm to (14.0, 21.6), turned to 0 degrees
- moved C3 6.84 mm to (48.3, 44.5)
- moved R18 3.81 mm to (34.3, 47.0)
- moved CLOCK_LED 3.59 mm to (11.4, 39.4), turned to 0 degrees
- moved CONTINUE_LED 3.59 mm to (40.6, 39.4), turned to 270 degrees
- moved R9 2.84 mm to (59.7, 26.7)
- moved LED1 2.84 mm to (59.7, 35.6), turned to 270 degrees
- moved R3 2.54 mm to (61.0, 53.3)
- moved R4 2.54 mm to (61.0, 44.5)
- moved START 2.54 mm to (19.1, 0.00)
- moved STOP_LED 2.54 mm to (38.1, 33.0)
- moved DIVISOR 2.54 mm to (73.7, 3.81)
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Connections:
- net N$1: now also U1.18; no longer U1.17
- net N$6: now also U1.17; no longer U1.18
Routing:
- net N$29: track 0.00 -> 313.1 mm
- net +5V: track 0.00 -> 294.8 mm
- net N$19: track 0.00 -> 151.5 mm
- net GND: track 0.00 -> 122.6 mm
- net +12V: track 0.00 -> 88.6 mm, vias 0 -> 2
- net N$31: track 0.00 -> 74.0 mm
- net N$30: track 0.00 -> 56.4 mm
- net N$1: track 0.00 -> 47.8 mm
- net N$17: track 0.00 -> 32.9 mm
- net N$10: track 0.00 -> 32.2 mm
- net N$22: track 0.00 -> 28.3 mm
- net N$9: track 0.00 -> 26.5 mm
- net N$11: track 0.00 -> 26.5 mm
- net N$6: track 0.00 -> 25.8 mm
- net N$23: track 0.00 -> 25.3 mm
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
Commit message: route tweaks
Parts:
- moved R19 2.54 mm to (34.3, 44.5)
- moved R3 1.91 mm to (62.9, 53.3)
- moved STOP_LED 1.27 mm to (39.4, 33.0)
- moved RST2 0.90 mm to (55.2, 62.9)
- moved RST1 0.64 mm to (55.2, 59.7)
Routing:
- net N$30: track 56.4 -> 54.0 mm
- net N$9: track 26.5 -> 24.6 mm
- net N$6: track 25.8 -> 24.1 mm
- net GND: track 122.6 -> 121.1 mm
- net N$1: track 47.8 -> 46.5 mm
- net N$29: track 313.1 -> 311.8 mm
- net N$19: track 151.5 -> 150.5 mm
- net N$7: track 16.5 -> 15.5 mm
- net +5V: track 294.8 -> 294.0 mm
- net +12V: track 88.6 -> 87.9 mm
- net N$43: track 7.34 -> 6.71 mm
- net N$3: track 9.81 -> 9.18 mm
- net N$39: track 7.33 -> 7.84 mm

Commit message: route tweaks
Parts:
- moved STOP_LED 1.27 mm to (40.6, 33.0)
- moved C1 1.27 mm to (38.1, 64.8)
- moved C3 0.90 mm to (47.6, 43.8)
- moved C2 0.64 mm to (22.9, 64.1)
Routing:
- net +5V: track 294.0 -> 297.5 mm
- net N$29: track 311.8 -> 308.4 mm
- net N$17: track 32.9 -> 35.2 mm
- net N$7: track 15.5 -> 13.5 mm
- net N$4: track 14.4 -> 12.7 mm
- net N$31: track 74.0 -> 75.1 mm
- net N$5: track 15.5 -> 14.5 mm
- net N$16: track 5.31 -> 4.49 mm
- net N$1: track 46.5 -> 45.8 mm
- net N$6: track 24.1 -> 24.8 mm
- net GND: track 121.1 -> 120.4 mm
- net N$19: track 150.5 -> 151.1 mm
- net N$13: track 9.07 -> 8.47 mm
- net +12V: track 87.9 -> 87.4 mm
- net N$40: track 11.5 -> 12.0 mm

Commit message: gcode
Parts:
- moved C3 1.42 mm to (47.0, 42.5)
- moved CLOCK_LED 1.27 mm to (10.2, 39.4)
- moved R18 0.64 mm to (34.3, 46.4)
- moved R19 0.64 mm to (34.3, 43.8)
Connections:
- removed net N$29: C1.1, C2.1, C3.2, C5.-, C8.2, CLOCK.P$1, CONTINUE.P$1, DIVISOR.1, OK1.5, PWR1.3, PWR1.4, PWR1.5, PWR1.6, PWR1.7, PWR1.8, RST2.1, START.P$1, STOP.P$1, U1.22, U1.8
- net GND: now also C1.1, C2.1, C3.2, C5.-, C8.2, CLOCK.P$1, CONTINUE.P$1, DIVISOR.1, OK1.5, PWR1.3, PWR1.4, PWR1.5, PWR1.6, PWR1.7, PWR1.8, RST2.1, START.P$1, STOP.P$1, U1.22, U1.8
Routing:
- net GND: track 120.4 -> 444.9 mm
- net N$29: track 308.4 -> 0.00 mm
- net +5V: track 297.5 -> 317.2 mm
- net N$19: track 151.1 -> 153.6 mm
- net N$17: track 35.2 -> 35.9 mm
- net N$1: track 45.8 -> 45.1 mm
- net N$39: track 7.84 -> 7.20 mm
- net N$40: track 12.0 -> 11.5 mm
- net N$9: track 24.4 -> 23.9 mm
Other:
- board size 100 x 80 mm -> 100 x 80.6 mm
